Commit message: working finally but the transition is not happening just start and end frames are being seen may revert back to this

File: robot.urdf (robot description, URDF)
Before this commit: robot simple_bot, 1 links, 0 joints
Links:
- added link base_footprint
- added link front_left_wheel; visual cylinder length=0.1 radius=0.15
- added link front_right_wheel; visual cylinder length=0.1 radius=0.15
- added link rear_left_wheel; visual cylinder length=0.1 radius=0.15
- added link rear_right_wheel; visual cylinder length=0.1 radius=0.15
- link base_link: geometry collision box size=1.0 0.6 0.3; visual box size=1.0 0.6 0.3
Joints:
- added joint base_joint: type fixed, parent base_footprint, child base_link, origin xyz=0 0 0.15 rpy=0 0 0
- added joint front_left_wheel_joint: type continuous, parent base_link, child front_left_wheel, origin xyz=0.3 0.35 -0.1 rpy=0 0 0, axis 0 1 0
- added joint front_right_wheel_joint: type continuous, parent base_link, child front_right_wheel, origin xyz=0.3 -0.35 -0.1 rpy=0 0 0, axis 0 1 0
- added joint rear_left_wheel_joint: type continuous, parent base_link, child rear_left_wheel, origin xyz=-0.3 0.35 -0.1 rpy=0 0 0, axis 0 1 0
- added joint rear_right_wheel_joint: type continuous, parent base_link, child rear_right_wheel, origin xyz=-0.3 -0.35 -0.1 rpy=0 0 0, axis 0 1 0
